File: STM32alt.kicad_pcb (KiCad board)
At the start: 2 copper layers, 26.7 x 76.2 mm, 27 parts, among them J3 USB_B, J4 Conn_01x04, J5 Conn_01x20, J6 Conn_02x03_Odd_Even, J7 Conn_01x02, J9 Conn_01x20, U1 LM1117-3.3, U2 STM32F103C8T6, Y1 8 MHz, Y2 Crystal

Commit message: Moved center chip, flipped SWD connector, added ground ring
Parts:
- moved J4 7.93 mm to (72.7, 33.8), turned to 270 degrees
- moved U2 0.31 mm to (68.9, 55.2)
Routing:
- net GNDB: track 109.8 -> 311.4 mm, vias 10 -> 98
- net 3V3B: track 116.1 -> 108.4 mm
- net PA13: track 42.6 -> 40.0 mm, vias 3 -> 2
- net PA14: track 29.9 -> 32.3 mm
- net PB5: track 5.38 -> 4.42 mm
- net PB7: track 6.83 -> 7.69 mm
- net PA4: track 5.17 -> 5.89 mm
- net PB8: track 9.69 -> 10.3 mm
- net PB9: track 11.3 -> 11.9 mm
- net PB2: track 15.3 -> 15.8 mm
